Commit message: multirobot urdf xacro

File: src/simulation/models/autogen/robot1.urdf (robot description, URDF)
Before this commit: robot turtlebot3_burger, 7 links, 6 joints
Links:
- removed link robot_1/base_footprint
- removed link robot_1/base_link
- removed link robot_1/base_scan
- removed link robot_1/caster_back_link
- removed link robot_1/imu_link
- removed link robot_1/wheel_left_link
- removed link robot_1/wheel_right_link
- added link robot1/base_footprint
- added link robot1/base_link, mass 8.2573504e-01; collision box size=0.140 0.140 0.143; visual mesh filename=src/simulation/models/turtlebot3_common/meshes/burger_base.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 scale=0.001 0.001 0.001
- added link robot1/base_scan, mass 0.114; collision cylinder length=0.0315 radius=0.055; visual mesh filename=src/simulation/models/turtlebot3_common/meshes/lds.dae scale=0.001 0.001 0.001
- added link robot1/caster_back_link, mass 0.005; collision box size=0.030 0.009 0.020
- added link robot1/imu_link
- added link robot1/wheel_left_link, mass 2.8498940e-02; collision cylinder length=0.018 radius=0.033; visual mesh filename=src/simulation/models/turtlebot3_common/meshes/tire.dae scale=0.001 0.001 0.001
- added link robot1/wheel_right_link, mass 2.8498940e-02; collision cylinder length=0.018 radius=0.033; visual mesh filename=src/simulation/models/turtlebot3_common/meshes/tire.dae scale=0.001 0.001 0.001
Joints:
- removed joint robot_1/caster_back_joint
- removed joint robot_1/imu_joint
- removed joint robot_1/scan_joint
- removed joint robot_1/wheel_left_joint
- removed joint robot_1/wheel_right_joint
- added joint caster_back_joint: type fixed, parent robot1/base_link, child robot1/caster_back_link, origin xyz=-0.081 0 -0.004 rpy=-1.57 0 0
- added joint imu_joint: type fixed, parent robot1/base_link, child robot1/imu_link, origin xyz=-0.032 0 0.068 rpy=0 0 0
- added joint scan_joint: type fixed, parent robot1/base_link, child robot1/base_scan, origin xyz=-0.032 0 0.172 rpy=0 0 0
- added joint wheel_left_joint: type continuous, parent robot1/base_link, child robot1/wheel_left_link, origin xyz=0.0 0.08 0.023 rpy=-1.57 0 0, axis 0 0 1
- added joint wheel_right_joint: type continuous, parent robot1/base_link, child robot1/wheel_right_link, origin xyz=0.0 -0.080 0.023 rpy=-1.57 0 0, axis 0 0 1
- joint base_joint: child robot_1/base_link -> robot1/base_link; parent robot_1/base_footprint -> robot1/base_footprint

File: src/simulation/models/autogen/robot2.urdf (robot description, URDF)
Before this commit: robot turtlebot3_burger, 7 links, 6 joints
Links:
- removed link robot_1/base_footprint
- removed link robot_1/base_link
- removed link robot_1/base_scan
- removed link robot_1/caster_back_link
- removed link robot_1/imu_link
- removed link robot_1/wheel_left_link
- removed link robot_1/wheel_right_link
- added link robot2/base_footprint
- added link robot2/base_link, mass 8.2573504e-01; collision box size=0.140 0.140 0.143; visual mesh filename=src/simulation/models/turtlebot3_common/meshes/burger_base.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 scale=0.001 0.001 0.001
- added link robot2/base_scan, mass 0.114; collision cylinder length=0.0315 radius=0.055; visual mesh filename=src/simulation/models/turtlebot3_common/meshes/lds.dae scale=0.001 0.001 0.001
- added link robot2/caster_back_link, mass 0.005; collision box size=0.030 0.009 0.020
- added link robot2/imu_link
- added link robot2/wheel_left_link, mass 2.8498940e-02; collision cylinder length=0.018 radius=0.033; visual mesh filename=src/simulation/models/turtlebot3_common/meshes/tire.dae scale=0.001 0.001 0.001
- added link robot2/wheel_right_link, mass 2.8498940e-02; collision cylinder length=0.018 radius=0.033; visual mesh filename=src/simulation/models/turtlebot3_common/meshes/tire.dae scale=0.001 0.001 0.001
Joints:
- removed joint robot_1/caster_back_joint
- removed joint robot_1/imu_joint
- removed joint robot_1/scan_joint
- removed joint robot_1/wheel_left_joint
- removed joint robot_1/wheel_right_joint
- added joint caster_back_joint: type fixed, parent robot2/base_link, child robot2/caster_back_link, origin xyz=-0.081 0 -0.004 rpy=-1.57 0 0
- added joint imu_joint: type fixed, parent robot2/base_link, child robot2/imu_link, origin xyz=-0.032 0 0.068 rpy=0 0 0
- added joint scan_joint: type fixed, parent robot2/base_link, child robot2/base_scan, origin xyz=-0.032 0 0.172 rpy=0 0 0
- added joint wheel_left_joint: type continuous, parent robot2/base_link, child robot2/wheel_left_link, origin xyz=0.0 0.08 0.023 rpy=-1.57 0 0, axis 0 0 1
- added joint wheel_right_joint: type continuous, parent robot2/base_link, child robot2/wheel_right_link, origin xyz=0.0 -0.080 0.023 rpy=-1.57 0 0, axis 0 0 1
- joint base_joint: child robot_1/base_link -> robot2/base_link; parent robot_1/base_footprint -> robot2/base_footprint

File: src/simulation/models/turtlebot3_burger.xacro (robot description, xacro)
@@ -1,7 +1,187 @@
 <robot xmlns:xacro="http://www.ros.org/wiki/xacro">
 <xacro:macro name="robot" params="ID">
-    <link name="base_link">
-    <origin xyz="0 0 0" rpy="0 0 0"/>
-    </link>
+  <!-- Init colour -->
+  <material name="black">
+      <color rgba="0.0 0.0 0.0 1.0"/>
+  </material>
+  <material name="dark">
+    <color rgba="0.3 0.3 0.3 1.0"/>
+  </material>
+  <material name="light_black">
+    <color rgba="0.4 0.4 0.4 1.0"/>
+  </material>
+  <material name="blue">
+    <color rgba="0.0 0.0 0.8 1.0"/>
+  </material>
+  <material name="green">
+    <color rgba="0.0 0.8 0.0 1.0"/>
+  </material>
+  <material name="grey">
+    <color rgba="0.5 0.5 0.5 1.0"/>
+  </material>
+  <material name="orange">
+    <color rgba="1.0 0.4235 0.0392 1.0"/>
+  </material>
+  <material name="brown">
+    <color rgba="0.8706 0.8118 0.7647 1.0"/>
+  </material>
+  <material name="red">
+    <color rgba="0.8 0.0 0.0 1.0"/>
+  </material>
+  <material name="white">
+    <color rgba="1.0 1.0 1.0 1.0"/>
+  </material>
+  <link name="robot${ID}/base_footprint"/>
+  <joint name="base_joint" type="fixed">
+    <parent link="robot${ID}/base_footprint"/>
+    <child link="robot${ID}/base_link"/>
+    <origin xyz="0.0 0.0 0.010" rpy="0 0 0"/>
+  </joint>
+  <link name="robot${ID}/base_link">
+    <visual>
+      <origin xyz="-0.032 0 0.0" rpy="0 0 0"/>
+      <geometry>
+        <mesh filename="src/simulation/models/turtlebot3_common/meshes/burger_base.dae" scale="0.001 0.001 0.001"/>
+      </geometry>
+      <material name="light_black"/>
+    </visual>
+    <collision>
+      <origin xyz="-0.032 0 0.070" rpy="0 0 0"/>
+      <geometry>
+        <box size="0.140 0.140 0.143"/>
+      </geometry>
+    </collision>
+    <inertial>
+      <origin xyz="0 0 0" rpy="0 0 0"/>
+      <mass value="8.2573504e-01"/>
+      <inertia ixx="2.2124416e-03" ixy="-1.2294101e-05" ixz="3.4938785e-05" iyy="2.1193702e-03" iyz="-5.0120904e-06" izz="2.0064271e-03" />
+    </inertial>
+  </link>
+  <joint name="wheel_left_joint" type="continuous">
+    <parent link="robot${ID}/base_link"/>
+    <child link="robot${ID}/wheel_left_link"/>
+    <origin xyz="0.0 0.08 0.023" rpy="-1.57 0 0"/>
+    <axis xyz="0 0 1"/>
+  </joint>
+  <link name="robot${ID}/wheel_left_link">
+    <visual>
+      <origin xyz="0 0 0" rpy="1.57 0 0"/>
+      <geometry>
+        <mesh filename="src/simulation/models/turtlebot3_common/meshes/tire.dae" scale="0.001 0.001 0.001"/>
+      </geometry>
+      <material name="dark"/>
+    </visual>
+    <collision>
+      <origin xyz="0 0 0" rpy="0 0 0"/>
+      <geometry>
+        <cylinder length="0.018" radius="0.033"/>
+      </geometry>
+    </collision>
+    <inertial>
+      <origin xyz="0 0 0" />
+      <mass value="2.8498940e-02" />
+      <inertia ixx="1.1175580e-05" ixy="-4.2369783e-11" ixz="-5.9381719e-09" iyy="1.1192413e-05" iyz="-1.4400107e-11" izz="2.0712558e-05" />
+    </inertial>
+  </link>
+  <joint name="wheel_right_joint" type="continuous">
+    <parent link="robot${ID}/base_link"/>
+    <child link="robot${ID}/wheel_right_link"/>
+    <origin xyz="0.0 -0.080 0.023" rpy="-1.57 0 0"/>
+    <axis xyz="0 0 1"/>
+  </joint>
+  <link name="robot${ID}/wheel_right_link">
+    <visual>
+      <origin xyz="0 0 0" rpy="1.57 0 0"/>
+      <geometry>
+        <mesh filename="src/simulation/models/turtlebot3_common/meshes/tire.dae" scale="0.001 0.001 0.001"/>
+      </geometry>
+      <material name="dark"/>
+    </visual>
+    <collision>
+      <origin xyz="0 0 0" rpy="0 0 0"/>
+      <geometry>
+        <cylinder length="0.018" radius="0.033"/>
+      </geometry>
+    </collision>
+    <inertial>
+      <origin xyz="0 0 0" />
+      <mass value="2.8498940e-02" />
+      <inertia ixx="1.1175580e-05" ixy="-4.2369783e-11" ixz="-5.9381719e-09" iyy="1.1192413e-05" iyz="-1.4400107e-11" izz="2.0712558e-05" />
+    </inertial>
+  </link>
+  <joint name="caster_back_joint" type="fixed">
+    <parent link="robot${ID}/base_link"/>
+    <child link="robot${ID}/caster_back_link"/>
+    <origin xyz="-0.081 0 -0.004" rpy="-1.57 0 0"/>
+  </joint>
+  <link name="robot${ID}/caster_back_link">
+    <collision>
+      <origin xyz="0 0.001 0" rpy="0 0 0"/>
+      <geometry>
+        <box size="0.030 0.009 0.020"/>
+      </geometry>
+    </collision>
+    <inertial>
+      <origin xyz="0 0 0" />
+      <mass value="0.005" />
+      <inertia ixx="0.001" ixy="0.0" ixz="0.0" iyy="0.001" iyz="0.0" izz="0.001" />
+    </inertial>
+  </link>
+  <joint name="imu_joint" type="fixed">
+    <parent link="robot${ID}/base_link"/>
+    <child link="robot${ID}/imu_link"/>
+    <origin xyz="-0.032 0 0.068" rpy="0 0 0"/>
+  </joint>
+  <link name="robot${ID}/imu_link"/>
+  <joint name="scan_joint" type="fixed">
+    <parent link="robot${ID}/base_link"/>
+    <child link="robot${ID}/base_scan"/>
+    <origin xyz="-0.032 0 0.172" rpy="0 0 0"/>
+  </joint>
+  <link name="robot${ID}/base_scan">
+    <visual>
+      <origin xyz="0 0 0.0" rpy="0 0 0"/>
+      <geometry>
+        <mesh filename="src/simulation/models/turtlebot3_common/meshes/lds.dae" scale="0.001 0.001 0.001"/>
+      </geometry>
+      <material name="dark"/>
+    </visual>
+    <collision>
+      <origin xyz="0.015 0 -0.0065" rpy="0 0 0"/>
+      <geometry>
+        <cylinder length="0.0315" radius="0.055"/>
+      </geometry>
+    </collision>
+    <inertial>
+      <mass value="0.114" />
+      <origin xyz="0 0 0" />
+      <inertia ixx="0.001" ixy="0.0" ixz="0.0" iyy="0.001" iyz="0.0" izz="0.001" />
+    </inertial>
+  </link>
+<gazebo>
+  <plugin name="diff_drive" filename="libgazebo_ros_diff_drive.so">
+            <ros>
+                <!--<namespace>/</namespace>-->
+            </ros>
+            <update_rate>30</update_rate>
+            <!-- wheels -->
+            <left_joint>wheel_left_joint</left_joint>
+            <right_joint>wheel_right_joint</right_joint>
+            <!-- kinematics -->
+            <wheel_separation>0.6855600</wheel_separation>
+            <wheel_diameter>0.4064000</wheel_diameter>
+            <!-- limits -->
+            <max_wheel_torque>20</max_wheel_torque>
+            <max_wheel_acceleration>1.0</max_wheel_acceleration>
+            <command_topic>robot${ID}/cmd_vel</command_topic>
+            <!-- output -->
+            <publish_odom>true</publish_odom>
+            <publish_odom_tf>true</publish_odom_tf>
+            <publish_wheel_tf>true</publish_wheel_tf>
+            <odometry_topic>robot${ID}/odom</odometry_topic>
+            <odometry_frame>robot${ID}/odom</odometry_frame>
+            <robot_base_frame>robot${ID}/base_footprint</robot_base_frame>
+        </plugin>
+        </gazebo>
 </xacro:macro>
 </robot>

Commit message: scan topics,mesh for all robots and tf2 fix

File: src/simulation/models/autogen/robot1.urdf (robot description, URDF)
Before this commit: robot turtlebot3_burger, 7 links, 6 joints
Links:
- link robot1/base_link: geometry collision box size=0.140 0.140 0.143; visual mesh filename=package://turtlebot3_gazebo/models/turtlebot3_common/meshes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 scale=0.001 0.001 0.001
- link robot1/base_scan: geometry collision cylinder length=0.0315 radius=0.055; visual mesh filename=package://turtlebot3_gazebo/models/turtlebot3_common/meshes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 scale=0.001 0.001 0.001
- link robot1/wheel_left_link: geometry collision cylinder length=0.018 radius=0.033; visual mesh filename=package://turtlebot3_gazebo/models/turtlebot3_common/meshes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 scale=0.001 0.001 0.001
- link robot1/wheel_right_link: geometry collision cylinder length=0.018 radius=0.033; visual mesh filename=package://turtlebot3_gazebo/models/turtlebot3_common/meshes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 scale=0.001 0.001 0.001
Joints:
- removed joint base_joint
- removed joint caster_back_joint
- removed joint imu_joint
- removed joint scan_joint
- removed joint wheel_left_joint
- removed joint wheel_right_joint
- added joint robot1/base_joint: type fixed, parent robot1/base_footprint, child robot1/base_link, origin xyz=0.0 0.0 0.010 rpy=0 0 0
- added joint robot1/caster_back_joint: type fixed, parent robot1/base_link, child robot1/caster_back_link, origin xyz=-0.081 0 -0.004 rpy=-1.57 0 0
- added joint robot1/imu_joint: type fixed, parent robot1/base_link, child robot1/imu_link, origin xyz=-0.032 0 0.068 rpy=0 0 0
- added joint robot1/scan_joint: type fixed, parent robot1/base_link, child robot1/base_scan, origin xyz=-0.032 0 0.172 rpy=0 0 0
- added joint robot1/wheel_left_joint: type continuous, parent robot1/base_link, child robot1/wheel_left_link, origin xyz=0.0 0.08 0.023 rpy=-1.57 0 0, axis 0 0 1
- added joint robot1/wheel_right_joint: type continuous, parent robot1/base_link, child robot1/wheel_right_link, origin xyz=0.0 -0.080 0.023 rpy=-1.57 0 0, axis 0 0 1

File: src/simulation/models/autogen/robot2.urdf (robot description, URDF)
Before this commit: robot turtlebot3_burger, 7 links, 6 joints
Links:
- link robot2/base_link: geometry collision box size=0.140 0.140 0.143; visual mesh filename=package://turtlebot3_gazebo/models/turtlebot3_common/meshes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 scale=0.001 0.001 0.001
- link robot2/base_scan: geometry collision cylinder length=0.0315 radius=0.055; visual mesh filename=package://turtlebot3_gazebo/models/turtlebot3_common/meshes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 scale=0.001 0.001 0.001
- link robot2/wheel_left_link: geometry collision cylinder length=0.018 radius=0.033; visual mesh filename=package://turtlebot3_gazebo/models/turtlebot3_common/meshes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 scale=0.001 0.001 0.001
- link robot2/wheel_right_link: geometry collision cylinder length=0.018 radius=0.033; visual mesh filename=package://turtlebot3_gazebo/models/turtlebot3_common/meshes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 scale=0.001 0.001 0.001
Joints:
- removed joint base_joint
- removed joint caster_back_joint
- removed joint imu_joint
- removed joint scan_joint
- removed joint wheel_left_joint
- removed joint wheel_right_joint
- added joint robot2/base_joint: type fixed, parent robot2/base_footprint, child robot2/base_link, origin xyz=0.0 0.0 0.010 rpy=0 0 0
- added joint robot2/caster_back_joint: type fixed, parent robot2/base_link, child robot2/caster_back_link, origin xyz=-0.081 0 -0.004 rpy=-1.57 0 0
- added joint robot2/imu_joint: type fixed, parent robot2/base_link, child robot2/imu_link, origin xyz=-0.032 0 0.068 rpy=0 0 0
- added joint robot2/scan_joint: type fixed, parent robot2/base_link, child robot2/base_scan, origin xyz=-0.032 0 0.172 rpy=0 0 0
- added joint robot2/wheel_left_joint: type continuous, parent robot2/base_link, child robot2/wheel_left_link, origin xyz=0.0 0.08 0.023 rpy=-1.57 0 0, axis 0 0 1
- added joint robot2/wheel_right_joint: type continuous, parent robot2/base_link, child robot2/wheel_right_link, origin xyz=0.0 -0.080 0.023 rpy=-1.57 0 0, axis 0 0 1

File: src/simulation/models/turtlebot3_burger.xacro (robot description, xacro)
@@ -33,5 +33,5 @@
   </material>
   <link name="robot${ID}/base_footprint"/>
-  <joint name="base_joint" type="fixed">
+  <joint name="robot${ID}/base_joint" type="fixed">
     <parent link="robot${ID}/base_footprint"/>
     <child link="robot${ID}/base_link"/>
@@ -42,6 +42,5 @@
       <origin xyz="-0.032 0 0.0" rpy="0 0 0"/>
       <geometry>
-        <mesh filename="src/simulation/models/turtlebot3_common/meshes/burger_base.dae" scale="0.001 0.001 0.001"/>
-      </geometry>
+        <mesh filename="package://turtlebot3_gazebo/models/turtlebot3_common/meshes/burger_base.dae" scale="0.001 0.001 0.001"/>      </geometry>
       <material name="light_black"/>
     </visual>
@@ -58,5 +57,5 @@
     </inertial>
   </link>
-  <joint name="wheel_left_joint" type="continuous">
+  <joint name="robot${ID}/wheel_left_joint" type="continuous">
     <parent link="robot${ID}/base_link"/>
     <child link="robot${ID}/wheel_left_link"/>
@@ -68,5 +67,5 @@
       <origin xyz="0 0 0" rpy="1.57 0 0"/>
       <geometry>
-        <mesh filename="src/simulation/models/turtlebot3_common/meshes/tire.dae" scale="0.001 0.001 0.001"/>
+        <mesh filename="package://turtlebot3_gazebo/models/turtlebot3_common/meshes/tire.dae" scale="0.001 0.001 0.001"/>
       </geometry>
       <material name="dark"/>
@@ -84,5 +83,5 @@
     </inertial>
   </link>
-  <joint name="wheel_right_joint" type="continuous">
+  <joint name="robot${ID}/wheel_right_joint" type="continuous">
     <parent link="robot${ID}/base_link"/>
     <child link="robot${ID}/wheel_right_link"/>
@@ -94,6 +93,6 @@
       <origin xyz="0 0 0" rpy="1.57 0 0"/>
       <geometry>
-        <mesh filename="src/simulation/models/turtlebot3_common/meshes/tire.dae" scale="0.001 0.001 0.001"/>
-      </geometry>
+        <mesh filename="package://turtlebot3_gazebo/models/turtlebot3_common/meshes/tire.dae" scale="0.001 0.001 0.001"/>
+              </geometry>
       <material name="dark"/>
     </visual>
@@ -110,5 +109,5 @@
     </inertial>
   </link>
-  <joint name="caster_back_joint" type="fixed">
+  <joint name="robot${ID}/caster_back_joint" type="fixed">
     <parent link="robot${ID}/base_link"/>
     <child link="robot${ID}/caster_back_link"/>
@@ -128,5 +127,5 @@
     </inertial>
   </link>
-  <joint name="imu_joint" type="fixed">
+  <joint name="robot${ID}/imu_joint" type="fixed">
     <parent link="robot${ID}/base_link"/>
     <child link="robot${ID}/imu_link"/>
@@ -134,5 +133,5 @@
   </joint>
   <link name="robot${ID}/imu_link"/>
-  <joint name="scan_joint" type="fixed">
+  <joint name="robot${ID}/scan_joint" type="fixed">
     <parent link="robot${ID}/base_link"/>
     <child link="robot${ID}/base_scan"/>
@@ -143,6 +142,6 @@
       <origin xyz="0 0 0.0" rpy="0 0 0"/>
       <geometry>
-        <mesh filename="src/simulation/models/turtlebot3_common/meshes/lds.dae" scale="0.001 0.001 0.001"/>
-      </geometry>
+        <mesh filename="package://turtlebot3_gazebo/models/turtlebot3_common/meshes/lds.dae" scale="0.001 0.001 0.001"/>
+        </geometry>
       <material name="dark"/>
     </visual>
@@ -158,4 +157,32 @@
       <inertia ixx="0.001" ixy="0.0" ixz="0.0" iyy="0.001" iyz="0.0" izz="0.001" />
     </inertial>
+    <gazebo reference="robot${ID}/base_scan">
+        <material>Gazebo/Red</material>
+        <sensor name="laser" type="ray">
+            <pose> 0 0 0 0 0 0 </pose>
+            <visualize>true</visualize>
+            <update_rate>10</update_rate>
+            <ray>
+                <scan>
+                    <horizontal>
+                        <samples>360</samples>
+                        <min_angle>-3.14</min_angle>
+                        <max_angle>3.14</max_angle>
+                    </horizontal>
+                </scan>
+                <range>
+                    <min>0.3</min>
+                    <max>12</max>
+                </range>
+            </ray>
+            <plugin name="laser_controller" filename="libgazebo_ros_ray_sensor.so">
+                <ros>
+                    <argument>~/out:=scan</argument>
+                </ros>
+                <output_type>sensor_msgs/LaserScan</output_type>
+                <frame_name>laser_frame</frame_name>
+            </plugin>
+        </sensor>
+    </gazebo>
   </link>
 <gazebo>
@@ -184,4 +211,15 @@
         </plugin>
         </gazebo>
+<gazebo>
+    <plugin name="turtlebot3_joint_state" filename="libgazebo_ros_joint_state_publisher.so">
+      <ros>
+        <!-- <namespace>/tb3</namespace> -->
+        <remapping>~/out:=robot${ID}/joint_states</remapping>
+      </ros>
+      <update_rate>30</update_rate>
+      <joint_name>robot${ID}/wheel_left_joint</joint_name>
+      <joint_name>robot${ID}/wheel_right_joint</joint_name>
+    </plugin>
+        </gazebo>
 </xacro:macro>
 </robot>
